File: hardware/fortunelabs_mainboard_v0/fortunelabs_mainboard_v0.kicad_sch (KiCad schematic)
At the start: 110 parts, among them J101 Barrel_Jack, J301 USB_C_Receptacle_USB2.0_14P, J401 Micro_SD_Card_Det_Hirose_DM3AT, J701 Conn_02x16_Odd_Even, J801 Conn_02x16_Odd_Even, J901 Conn_02x07_Odd_Even, Q101 AO3401A, SW101 BOOT, SW102 RESET, U101 TPS62162DSG, U201 ESP32-S3-WROOM-2, U501 DS3232M, U601 TPL5010, U701 MCP23017_ML, U801 ADS1115, U802 ADS1115, U901 ULN2803A

Commit message: hw(hardware): change BT1 to the Keystone 1058 footprint
BT1 was BatteryHolder_Keystone_3002_1x2032; it is now
BatteryHolder_Keystone_1058_1x2032. Both take a 1x2032 cell, but the
1058 is a retainer clip rather than a holder, so the land pattern
differs.

The PCB has not been re-synced from the schematic and still carries the
3002 footprint. That update is left for its own commit.
Parts:
- BT1: footprint Battery:BatteryHolder_Keystone_3002_1x2032 -> Battery:BatteryHolder_Keystone_1058_1x2032
Changed lines of the file:
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@@
 			)
 		)
-		(property "Footprint" "Battery:BatteryHolder_Keystone_3002_1x2032"
+		(property "Footprint" "Battery:BatteryHolder_Keystone_1058_1x2032"
 			(at 54.864 179.07 90)
 			(effects
